Commit message: rename stl files, update cmake lists

File: src/xela_hand_controllers/urdf/my_xela_allegro.urdf (robot description, URDF)
Before this commit: robot allegro_hand_right, 44 links, 43 joints
Links:
- link index_link_1: geometry collision box size=0.0196 0.0275 0.0164; visual mesh filename=package://xela_hand_controllers/mesh/allegro/link_0_ext.stl
- link index_link_4: geometry collision box size=0.0196 0.0275 0.026399999999999996; visual mesh filename=package://xela_hand_controllers/mesh/allegro/link_3.stl
- link middle_link_1: geometry collision box size=0.0196 0.0275 0.0164; visual mesh filename=package://xela_hand_controllers/mesh/allegro/link_0_ext.stl
- link middle_link_4: geometry collision box size=0.0196 0.0275 0.026399999999999996; visual mesh filename=package://xela_hand_controllers/mesh/allegro/link_3.stl
- link ring_link_1: geometry collision box size=0.0196 0.0275 0.0164; visual mesh filename=package://xela_hand_controllers/mesh/allegro/link_0_ext.stl
- link ring_link_4: geometry collision box size=0.0196 0.0275 0.026399999999999996; visual mesh filename=package://xela_hand_controllers/mesh/allegro/link_3.stl
- link thumb_link_2: geometry collision box size=0.0196 0.0275 0.0177; visual mesh filename=package://xela_hand_controllers/mesh/allegro/link_0_ext.stl
